File: 60-xt-pcb.kicad_pcb (KiCad board)
At the start: 2 copper layers, 171 parts, among them J1 Conn_01x04, Q1 2N7002, SW1 SW_Push, U1 MCP1700-3302E_SOT23, U2 STM32F072CBTx

Commit message: finish routing, add logos
Parts:
- added LOGO1: O-LOGO, board_logos:o-logo-300dpi, F.Cu at (293.7, 162.7)
- added LOGO2: O-LOGO, board_logos:o-logo-back-300dpi, F.Cu at (236.5, 162.7)
- C1, C10, C11, C12, C2, C3, C4, C5, C6, C7, C8, C9, D1, D2, F1, Q1, R1, R2, R3, R4, U1, U2: moved to B.Cu
- moved F1 164.0 mm to (120.4, 139.1), turned to 270 degrees
- moved U1 161.1 mm to (121.9, 122.7), turned to 90 degrees
- moved D1 159.6 mm to (125.3, 127.4), turned to 90 degrees
- moved D2 155.5 mm to (121.8, 133.1), turned to 180 degrees
- moved C12 152.1 mm to (150.0, 102.7), turned to 180 degrees
- moved C2 142.6 mm to (125.3, 122.9), turned to 90 degrees
- moved Q1 139.2 mm to (151.8, 136.6)
- moved C5 131.3 mm to (145.4, 104.0), turned to 180 degrees
- moved C1 131.0 mm to (121.7, 125.7)
- moved C6 125.7 mm to (143.6, 106.2), turned to 180 degrees
- moved R1 125.6 mm to (151.6, 132.3), turned to 180 degrees
- moved R4 125.5 mm to (143.3, 132.9), turned to 90 degrees
- moved R2 123.8 mm to (148.4, 134.4)
- moved C11 118.6 mm to (150.0, 104.4), turned to 180 degrees
- moved C7 115.1 mm to (143.8, 116.5), turned to 270 degrees
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Connections:
- U2 pad 13: Net-(U2-Pad13) -> Col3
- U2 pad 14: Net-(U2-Pad14) -> Col15
- U2 pad 15: Net-(U2-Pad15) -> Col14
- U2 pad 16: Net-(U2-Pad16) -> Col13
- U2 pad 17: Net-(U2-Pad17) -> Col12
- U2 pad 18: Net-(U2-Pad18) -> Col11
- U2 pad 19: Net-(U2-Pad19) -> Col10
- U2 pad 20: Net-(U2-Pad20) -> Col9
- U2 pad 21: Net-(U2-Pad21) -> Col8
- U2 pad 22: Net-(U2-Pad22) -> Col7
- U2 pad 25: Net-(U2-Pad25) -> Col6
- U2 pad 26: Net-(U2-Pad26) -> Col5
- U2 pad 27: Net-(U2-Pad27) -> Col4
- U2 pad 31: Net-(U2-Pad31) -> CAPS
- U2 pad 39: Net-(U2-Pad39) -> Col2
- U2 pad 40: Net-(U2-Pad40) -> Row2
- U2 pad 41: Net-(U2-Pad41) -> Col1
- U2 pad 42: Net-(U2-Pad42) -> Col0
- U2 pad 43: Net-(U2-Pad43) -> Row3
- U2 pad 45: Net-(U2-Pad45) -> Row4
- U2 pad 46: Net-(U2-Pad46) -> Row0
- U2 pad 5: Net-(U2-Pad5) -> Row1
Routing:
- net Row4: track 0.00 -> 407.7 mm, vias 0 -> 2
- net Row3: track 0.00 -> 374.7 mm, vias 0 -> 2
- net Col15: track 0.00 -> 342.4 mm, vias 0 -> 1
- net Row0: track 0.00 -> 341.3 mm, vias 0 -> 2
- net Row2: track 0.00 -> 340.9 mm, vias 0 -> 2
- net Col14: track 0.00 -> 325.1 mm
- net Row1: track 0.00 -> 323.5 mm
- net Col13: track 0.00 -> 291.3 mm
- net Col12: track 0.00 -> 270.5 mm
- net Col11: track 0.00 -> 232.2 mm
- net Col10: track 0.00 -> 212.9 mm
- net Col8: track 0.00 -> 195.2 mm
- net Col9: track 0.00 -> 193.7 mm
- net Col7: track 0.00 -> 155.2 mm
- net GND: track 0.00 -> 154.4 mm, vias 0 -> 6
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- added copper zone on B.Cu, net GND
Other:
- board outline added: 327.1 x 93.8 mm
